File: src/kicad/rpi-rgb-led-matrix-ji/rpi-rgb-led-matrix-nonhat.kicad_pcb (KiCad board)
At the start: 2 copper layers, 65 x 56 mm, 40 parts, among them J3 Screw_Terminal_01x02, J4 Conn_02x08_Odd_Even, J5 Conn_02x08_Odd_Even, J6 Conn_02x08_Odd_Even, J7 Header_2x3, J8 Header_2x4, P1 Raspberry_Pi_2_3, Q1 DMG2305UX, Q2 DMMT5401, U1 74HCT245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

Commit message: m
Routing:
- net +5VP: track 23.4 -> 25.9 mm, vias 1 -> 3
- net +5V: track 119.2 -> 117.6 mm
- net Net-(R1-Pad2): track 72.4 -> 71.4 mm
- net GND: vias 15 -> 19
Other:
- board text added: "Bug: solder jumpers report pads too close in DRC. Ignore the complaints on the solder jumpers."
- board text removed: "Bug: bridged solder jumpers report pads too close in DRC. Ignore the complaints on the solder jumpers."
